Commit message: Fixes

File: dbw_mkz_description/urdf/mkz.urdf.xacro (robot description, xacro)
@@ -48,5 +48,5 @@
         <origin xyz="0 0.002 0" rpy="0 ${-M_PI/2 + flip*M_PI} 0"/>
         <geometry>
-          <mesh filename="package://mkz_description/meshes/wheel.dae" scale="1 1 1" />
+          <mesh filename="package://dbw_mkz_description/meshes/wheel.dae" scale="1 1 1" />
         </geometry>
       </visual>
@@ -64,5 +64,5 @@
         <origin xyz="0 0.002 0" rpy="0 ${-M_PI/2 + flip*M_PI} 0"/>
         <geometry>
-          <mesh filename="package://mkz_description/meshes/wheel.dae" scale="1 1 1" />
+          <mesh filename="package://dbw_mkz_description/meshes/wheel.dae" scale="1 1 1" />
         </geometry>
       </visual>
@@ -81,5 +81,5 @@
       <origin xyz="0 0 -0.3323" rpy="0 0 ${M_PI/2}" />
       <geometry>
-        <mesh filename="package://mkz_description/meshes/body.dae" />
+        <mesh filename="package://dbw_mkz_description/meshes/body.dae" />
       </geometry>
     </visual>

Commit message: Added Gazebo simulation model to dbw_mkz_description, maintaining backward compatibility.

File: dbw_mkz_description/urdf/mkz.urdf.xacro (robot description, xacro)
@@ -1,93 +1,4 @@
 <?xml version="1.0"?>
 <robot name="mobility_base" xmlns:xacro="http://www.ros.org/wiki/xacro" >
-  <xacro:property name="M_PI" value="3.1415926535897931" />
-  <xacro:property name="wheel_base_x" value="${2.8448}" />
-  <xacro:property name="wheel_base_y" value="${1.5748/2}" />
-  <xacro:property name="wheel_radius" value="0.2413" />
-  <!-- Materials -->
-  <xacro:macro name="darkred_material" >
-    <material name="darkred" >
-      <color rgba=".5 .1 .1 1"/>
-    </material>
-  </xacro:macro>
-  <xacro:macro name="grey_material" >
-    <material name="grey" >
-      <color rgba=".5 .5 .5 1"/>
-    </material>
-  </xacro:macro>
-  <xacro:macro name="black_material" >
-    <material name="black" >
-      <color rgba=".1 .1 .1 1"/>
-    </material>
-  </xacro:macro>
-  <xacro:macro name="steering" params="suffix reflecty" >
-    <link name="steer${suffix}" >
-      <inertial>
-        <mass value="1" />
-        <inertia ixx="1.0" ixy="0.0" ixz="0.0"
-          iyx="0.0" iyy="1.0" iyz="0.0"
-          izx="0.0" izy="0.0" izz="1.0" />
-      </inertial>
-    </link>
-    <joint name="steer${suffix}" type="continuous" >
-      <parent link="base_link" />
-      <child link="steer${suffix}" />
-      <origin xyz="${wheel_base_x} ${reflecty*wheel_base_y} 0" rpy="0 0 0" />
-      <axis xyz="0 0 1" />
-    </joint>
-  </xacro:macro>
-  <xacro:macro name="front_wheel" params="suffix reflectx reflecty flip" >
-    <joint name="wheel${suffix}" type="continuous" >
-      <parent link="steer${suffix}" />
-      <child link="wheel${suffix}" />
-      <origin xyz="0 0 0" rpy="${-M_PI/2} 0 0" />
-      <axis xyz="0 0 1" />
-    </joint>
-    <link name="wheel${suffix}" >
-      <visual>
-        <origin xyz="0 0.002 0" rpy="0 ${-M_PI/2 + flip*M_PI} 0"/>
-        <geometry>
-          <mesh filename="package://dbw_mkz_description/meshes/wheel.dae" scale="1 1 1" />
-        </geometry>
-      </visual>
-    </link>
-  </xacro:macro>
-  <xacro:macro name="rear_wheel" params="suffix reflectx reflecty flip" >
-    <joint name="wheel${suffix}" type="continuous" >
-      <parent link="base_link" />
-      <child link="wheel${suffix}" />
-      <origin xyz="${reflectx*wheel_base_x} ${reflecty*wheel_base_y} 0" rpy="${-M_PI/2} 0 0" />
-      <axis xyz="0 0 1" />
-    </joint>
-    <link name="wheel${suffix}" >
-      <visual>
-        <origin xyz="0 0.002 0" rpy="0 ${-M_PI/2 + flip*M_PI} 0"/>
-        <geometry>
-          <mesh filename="package://dbw_mkz_description/meshes/wheel.dae" scale="1 1 1" />
-        </geometry>
-      </visual>
-    </link>
-  </xacro:macro>
-  <!-- Base Footprint -->
-  <link name="base_footprint" />
-  <!-- Base Link -->
-  <joint name="footprint" type="fixed" >
-   <parent link="base_footprint" />
-    <child link="base_link" />
-    <origin xyz="0 0 ${wheel_radius+0.09}" rpy="0 0 0" />
-  </joint>
-  <link name="base_link" >
-    <visual>
-      <origin xyz="0 0 -0.3323" rpy="0 0 ${M_PI/2}" />
-      <geometry>
-        <mesh filename="package://dbw_mkz_description/meshes/body.dae" />
-      </geometry>
-    </visual>
-  </link>
-  <xacro:front_wheel suffix="_fl" reflectx=" 1" reflecty=" 1" flip="0" />
-  <xacro:front_wheel suffix="_fr" reflectx=" 1" reflecty=" -1" flip="1" />
-  <xacro:rear_wheel suffix="_rl" reflectx=" 0" reflecty=" 1" flip="0" />
-  <xacro:rear_wheel suffix="_rr" reflectx=" 0" reflecty=" -1" flip="1" />
-  <xacro:steering suffix="_fl" reflecty=" 1" />
-  <xacro:steering suffix="_fr" reflecty=" -1" />
+  <xacro:include filename="$(find dbw_mkz_description)/urdf/mkz_structure.urdf.xacro" />
 </robot>

Commit message: Added 2017 MKZ, 2013 - 2017 Fusion, and 2013 - 2017 Mondeo URDF models.

File: dbw_mkz_description/urdf/mkz.urdf.xacro (robot description, xacro)
@@ -1,4 +1,4 @@
 <?xml version="1.0"?>
-<robot name="mobility_base" xmlns:xacro="http://www.ros.org/wiki/xacro" >
-  <xacro:include filename="$(find dbw_mkz_description)/urdf/mkz_structure.urdf.xacro" />
+<robot name="mkz" xmlns:xacro="http://www.ros.org/wiki/xacro" >
+  <xacro:include filename="$(find dbw_mkz_description)/urdf/mkz_13_structure.urdf.xacro" />
 </robot>

File: dbw_mkz_description/urdf/mkz_17_structure.urdf.xacro (robot description, xacro)
@@ -1,41 +1,29 @@
 <?xml version="1.0"?>
-<robot name="dbw_mkz" xmlns:xacro="http://www.ros.org/wiki/xacro">
-  <xacro:arg name="dae_file" default="$(find dbw_mkz_description)/meshes/body.dae"/>
+<!-- created with Phobos 0.7 -->
+  <robot name="dbw_mkz" xmlns:xacro="http://www.ros.org/wiki/xacro">
+    <xacro:arg name="dae_file" default="$(find dbw_mkz_description)/meshes/mkz_13/body.dae"/>
     <link name="base_footprint">
     </link>
     <link name="base_link">
       <inertial>
-        <origin xyz="0 0 0.071011" rpy="0 0 0"/>
+        <origin xyz="0 0 0.25" rpy="0 0 0"/>
         <mass value="1500.0"/>
         <inertia ixx="1000.0" ixy="0" ixz="0" iyy="1000.0" iyz="0" izz="1000.0"/>
       </inertial>
-      <visual name="Raw Windshield">
-        <origin xyz="0.667205 0 0.859831" rpy="0 0 1.570796"/>
+      <visual name="chassis">
+        <origin xyz="-0.032498 0 -0.371498" rpy="0 0 1.570796"/>
         <geometry>
-          <mesh filename="package://dbw_mkz_description/meshes/windshield.dae" scale="1.0 1.0 1.0"/>
+          <mesh filename="file://$(arg dae_file)" scale="1 0.964 1"/>
         </geometry>
-      </visual>
-      <visual name="Raw_Back_Window">
-        <origin xyz="-1.466892 0 0.926" rpy="0 0 -1.570796"/>
-        <geometry>
-          <mesh filename="package://dbw_mkz_description/meshes/back_window.dae" scale="1.0 1.0 1.0"/>
-        </geometry>
-        <material name="Material_001.001"/>
-      </visual>
-      <visual name="chassis">
-        <origin xyz="-0.04 0 -0.33" rpy="0 0 1.570796"/>
-        <geometry>
-          <mesh filename="file://$(arg dae_file)" scale="0.01 0.01 0.01"/>
-        </geometry>
-        <material name="roof"/>
+        <material name="black.001"/>
       </visual>
       <collision name="chassis_collision">
-        <origin xyz="0.084967 -0.03046 0.350609" rpy="1.570796 0 -3.141593"/>
+        <origin xyz="0.054381 -0.019748 0.332734" rpy="1.570796 0 -3.141593"/>
         <geometry>
-          <mesh filename="package://dbw_mkz_description/meshes/mkz_collision.stl" scale="0.001 0.001 0.001"/>
+          <mesh filename="package://dbw_mkz_description/meshes/body_collision.stl" scale="0.001 0.001 0.001"/>
         </geometry>
       </collision>
     </link>
-    <link name="left_steer">
+    <link name="steer_fl">
       <inertial>
         <origin xyz="-0.013054 -0.0295 0" rpy="0 0 0"/>
@@ -44,5 +32,5 @@
       </inertial>
     </link>
-    <link name="right_steer">
+    <link name="steer_fr">
       <inertial>
         <origin xyz="-0.01305 0.0275 0" rpy="0 0 0"/>
@@ -58,9 +46,9 @@
       </inertial>
       <visual name="wheel_fl_visual">
-        <origin xyz="0.0004 -0.005 0.0775" rpy="-1.570796 -1.570796 0"/>
+        <origin xyz="-0.0026 0 0.017813" rpy="-1.570796 1.570796 0"/>
         <geometry>
-          <mesh filename="package://dbw_mkz_description/meshes/wheel.dae" scale="0.01 0.01 0.01"/>
+          <mesh filename="package://dbw_mkz_description/meshes/mkz_17/wheel.dae" scale="0.01 0.01 0.01"/>
         </geometry>
-        <material name="tire_001.001"/>
+        <material name="carpaint_002"/>
       </visual>
       <collision name="wheel_fl_collision">
@@ -78,12 +66,12 @@
       </inertial>
       <visual name="wheel_fr_visual">
-        <origin xyz="0.0004 -0.005 -0.0775" rpy="-1.570796 1.570796 0"/>
+        <origin xyz="-0.0026 0 -0.0217" rpy="-1.570796 -1.570796 0"/>
         <geometry>
-          <mesh filename="package://dbw_mkz_description/meshes/wheel.dae" scale="0.01 0.01 0.01"/>
+          <mesh filename="package://dbw_mkz_description/meshes/mkz_17/wheel.dae" scale="0.01 0.01 0.01"/>
         </geometry>
-        <material name="tire_001.002"/>
+        <material name="carpaint_002.001"/>
       </visual>
       <collision name="wheel_fr_collision">
-        <origin xyz="0 0 0" rpy="0 3.141593 0"/>
+        <origin xyz="0 0 -0.0035" rpy="0 3.141593 0"/>
         <geometry>
           <cylinder radius="0.33" length="0.2"/>
@@ -98,9 +86,9 @@
       </inertial>
       <visual name="wheel_rl_visual">
-        <origin xyz="-0.0004 -0.005 0.056382" rpy="-1.570796 -1.570796 0"/>
+        <origin xyz="0.0026 0 -0.00412" rpy="-1.570796 1.570796 0"/>
         <geometry>
-          <mesh filename="package://dbw_mkz_description/meshes/wheel.dae" scale="0.01 0.01 0.01"/>
+          <mesh filename="package://dbw_mkz_description/meshes/mkz_17/wheel.dae" scale="0.01 0.01 0.01"/>
         </geometry>
-        <material name="tire_001"/>
+        <material name="carpaint_002.003"/>
       </visual>
       <collision name="wheel_rl_collision">
@@ -118,9 +106,9 @@
       </inertial>
       <visual name="wheel_rr_visual">
-        <origin xyz="-0.0004 -0.005 -0.057" rpy="-1.570796 1.570796 0"/>
+        <origin xyz="0.0026 0 0.00331" rpy="-1.570796 -1.570796 0"/>
         <geometry>
-          <mesh filename="package://dbw_mkz_description/meshes/wheel.dae" scale="0.01 0.01 0.01"/>
+          <mesh filename="package://dbw_mkz_description/meshes/mkz_17/wheel.dae" scale="0.01 0.01 0.01"/>
         </geometry>
-        <material name="tire_001.003"/>
+        <material name="carpaint_002.002"/>
       </visual>
       <collision name="wheel_rr_collision">
@@ -136,15 +124,15 @@
       <child link="base_link"/>
     </joint>
-    <joint name="left_steer" type="revolute">
+    <joint name="steer_fl" type="revolute">
       <origin xyz="1.435054 0.817 0.33" rpy="0 0 0"/>
       <parent link="base_link"/>
-      <child link="left_steer"/>
+      <child link="steer_fl"/>
       <axis xyz="0 0 1.0"/>
       <limit lower="-0.6" upper="0.6" effort="0" velocity="0"/>
     </joint>
-    <joint name="right_steer" type="revolute">
+    <joint name="steer_fr" type="revolute">
       <origin xyz="1.43505 -0.815 0.33" rpy="0 0 0"/>
       <parent link="base_link"/>
-      <child link="right_steer"/>
+      <child link="steer_fr"/>
       <axis xyz="0 0 1.0"/>
       <limit lower="-0.6" upper="0.6" effort="0" velocity="0"/>
@@ -152,5 +140,5 @@
     <joint name="wheel_fl" type="continuous">
       <origin xyz="-0.012654 -0.0295 -0.33" rpy="1.570796 0 -3.141593"/>
-      <parent link="left_steer"/>
+      <parent link="steer_fl"/>
       <child link="wheel_fl"/>
       <axis xyz="0 0 1.0"/>
@@ -159,5 +147,5 @@
     <joint name="wheel_fr" type="continuous">
       <origin xyz="-0.01265 0.0275 -0.33" rpy="1.570796 0 -3.141593"/>
-      <parent link="right_steer"/>
+      <parent link="steer_fr"/>
       <child link="wheel_fr"/>
       <axis xyz="0 0 1.0"/>
@@ -178,21 +166,18 @@
       <limit effort="5000.0" velocity="22.0"/>
     </joint>
-    <material name="Material_001.001">
-      <color rgba="0.64 0.64 0.64 1.0"/>
+    <material name="black.001">
+      <color rgba="0 0 0 1.0"/>
     </material>
-    <material name="roof">
-      <color rgba="0.48 0.48 0.48 1.0"/>
+    <material name="carpaint_002">
+      <color rgba="0.941177 0.941177 0.941177 1.0"/>
     </material>
-    <material name="tire_001">
-      <color rgba="0.084706 0.084706 0.084706 1.0"/>
+    <material name="carpaint_002.001">
+      <color rgba="0.941177 0.941177 0.941177 1.0"/>
     </material>
-    <material name="tire_001.001">
-      <color rgba="0.084706 0.084706 0.084706 1.0"/>
+    <material name="carpaint_002.002">
+      <color rgba="0.941177 0.941177 0.941177 1.0"/>
     </material>
-    <material name="tire_001.002">
-      <color rgba="0.084706 0.084706 0.084706 1.0"/>
+    <material name="carpaint_002.003">
+      <color rgba="0.941177 0.941177 0.941177 1.0"/>
     </material>
-    <material name="tire_001.003">
-      <color rgba="0.084706 0.084706 0.084706 1.0"/>
-    </material>
-</robot>
+  </robot>

File: dbw_mkz_description/urdf/vehicle_gazebo.urdf.xacro (robot description, xacro)
@@ -1,5 +1,5 @@
 <?xml version="1.0"?>
 <robot name="mkz_gazebo" xmlns:xacro="http://www.ros.org/wiki/xacro">
-  <xacro:property name="wheel_friction" value="0.8" />
+  <xacro:property name="wheel_friction" value="1.2" />
   <xacro:arg name="pub_odom" default="false"/>
   <xacro:arg name="pub_tf" default="false"/>
@@ -26,16 +26,10 @@
   <gazebo>
     <!-- Simulated vehicle interface -->
-    <plugin name="mkz_interface_plugin" filename="libdbw_mkz_gazebo_vehicle.so" >
+    <plugin name="dbw_interface_plugin" filename="libdbw_mkz_gazebo_vehicle.so" >
       <start_gear>$(arg start_gear)</start_gear>
+      <car_model>$(arg car_model)</car_model>
+      <car_year>$(arg car_year)</car_year>
     </plugin>
-    <!-- Publish joint states -->
-    <plugin name="joint_state_publisher" filename="libgazebo_ros_joint_state_publisher.so">
-        <jointName>
-            left_steer, right_steer, wheel_fl, wheel_fr, wheel_rl, wheel_rr
-        </jointName>
-        <updateRate>100</updateRate>
-        <alwaysOn>true</alwaysOn>
-    </plugin>
-    <!-- Publish TF and twist measurements -->
+    <!-- Publish TF and odom messages with true global frame pose and velocity -->
     <plugin name="pose_plugin" filename="libdbw_mkz_gazebo_pose.so" >
       <pub_tf>$(arg pub_tf)</pub_tf>

File: dbw_mkz_description/urdf/vehicle_sensors.urdf.xacro (robot description, xacro)
@@ -1,5 +1,5 @@
 <?xml version="1.0"?>
 <robot name="mkz_sensors" xmlns:xacro="http://www.ros.org/wiki/xacro" >
-  <xacro:macro name="mkz_camera" params="name parent_link x y z roll pitch yaw" >
+  <xacro:macro name="dbw_mkz_camera" params="name parent_link x y z roll pitch yaw" >
     <link name="${name}" >
       <visual>
@@ -64,5 +64,5 @@
     </gazebo>
   </xacro:macro>
-  <xacro:macro name="mkz_gps" params="name parent_link x y z roll pitch yaw rate ref_lat ref_lon" >
+  <xacro:macro name="dbw_mkz_gps" params="name parent_link x y z rate ref_lat ref_lon" >
     <link name="${name}" >
       <visual>
