Commit message: Added year to fusion and mondeo mesh and model names.

File: dbw_mkz_description/urdf/fusion_13_structure.urdf.xacro (robot description, xacro)
@@ -2,5 +2,5 @@
 <!-- created with Phobos 0.7 -->
   <robot name="dbw_mkz" xmlns:xacro="http://www.ros.org/wiki/xacro">
-    <xacro:arg name="dae_file" default="$(find dbw_mkz_description)/meshes/mondeo/body.dae"/>
+    <xacro:arg name="dae_file" default="$(find dbw_mkz_description)/meshes/mkz_13/body.dae"/>
     <link name="base_footprint">
     </link>
@@ -12,14 +12,14 @@
       </inertial>
       <visual name="chassis">
-        <origin xyz="-0.061355 0 -0.33647" rpy="0 0 1.570796"/>
+        <origin xyz="-0.045056 0 -0.373676" rpy="0 0 1.570796"/>
         <geometry>
-          <mesh filename="file://$(arg dae_file)" scale="1 1 1"/>
+          <mesh filename="file://$(arg dae_file)" scale="1 0.964 1"/>
         </geometry>
         <material name="black.001"/>
       </visual>
       <collision name="chassis_collision">
-        <origin xyz="0.039687 -0.03046 0.350609" rpy="1.570796 0 -3.141593"/>
+        <origin xyz="0.058756 -0.03046 0.325149" rpy="1.570796 0 -3.141593"/>
         <geometry>
-          <mesh filename="package://dbw_mkz_description/meshes/body_collision.stl" scale="0.001 0.001 0.001"/>
+          <mesh filename="package://dbw_mkz_description/meshes/body_collision.stl" scale="0.000965 0.001 0.001"/>
         </geometry>
       </collision>
@@ -46,7 +46,7 @@
       </inertial>
       <visual name="wheel_fl_visual">
-        <origin xyz="-0.0026 0 0.032213" rpy="-1.570796 1.570796 0"/>
+        <origin xyz="0 0 0.0385" rpy="-1.570796 -1.570796 0"/>
         <geometry>
-          <mesh filename="package://dbw_mkz_description/meshes/mondeo/wheel.dae" scale="0.01 0.01 0.01"/>
+          <mesh filename="package://dbw_mkz_description/meshes/fusion_13/wheel.dae" scale="0.01 0.01 0.01"/>
         </geometry>
         <material name="carpaint_002"/>
@@ -66,7 +66,7 @@
       </inertial>
       <visual name="wheel_fr_visual">
-        <origin xyz="-0.0026 0 -0.035355" rpy="-1.570796 -1.570796 0"/>
+        <origin xyz="0 0 -0.043777" rpy="-1.570796 1.570796 0"/>
         <geometry>
-          <mesh filename="package://dbw_mkz_description/meshes/mondeo/wheel.dae" scale="0.01 0.01 0.01"/>
+          <mesh filename="package://dbw_mkz_description/meshes/fusion_13/wheel.dae" scale="0.01 0.01 0.01"/>
         </geometry>
         <material name="carpaint_002.001"/>
@@ -86,7 +86,7 @@
       </inertial>
       <visual name="wheel_rl_visual">
-        <origin xyz="0.0026 0 0.010943" rpy="-1.570796 1.570796 0"/>
+        <origin xyz="0 0 0.017382" rpy="-1.570796 -1.570796 0"/>
         <geometry>
-          <mesh filename="package://dbw_mkz_description/meshes/mondeo/wheel.dae" scale="0.01 0.01 0.01"/>
+          <mesh filename="package://dbw_mkz_description/meshes/fusion_13/wheel.dae" scale="0.01 0.01 0.01"/>
         </geometry>
         <material name="carpaint_002.003"/>
@@ -106,7 +106,7 @@
       </inertial>
       <visual name="wheel_rr_visual">
-        <origin xyz="0.0026 0 -0.010783" rpy="-1.570796 -1.570796 0"/>
+        <origin xyz="0 0 -0.019214" rpy="-1.570796 1.570796 0"/>
         <geometry>
-          <mesh filename="package://dbw_mkz_description/meshes/mondeo/wheel.dae" scale="0.01 0.01 0.01"/>
+          <mesh filename="package://dbw_mkz_description/meshes/fusion_13/wheel.dae" scale="0.01 0.01 0.01"/>
         </geometry>
         <material name="carpaint_002.002"/>

File: dbw_mkz_description/urdf/mondeo_15_structure.urdf.xacro (robot description, xacro)
@@ -2,5 +2,5 @@
 <!-- created with Phobos 0.7 -->
   <robot name="dbw_mkz" xmlns:xacro="http://www.ros.org/wiki/xacro">
-    <xacro:arg name="dae_file" default="$(find dbw_mkz_description)/meshes/mkz_13/body.dae"/>
+    <xacro:arg name="dae_file" default="$(find dbw_mkz_description)/meshes/mondeo/body.dae"/>
     <link name="base_footprint">
     </link>
@@ -12,14 +12,14 @@
       </inertial>
       <visual name="chassis">
-        <origin xyz="-0.045056 0 -0.373676" rpy="0 0 1.570796"/>
+        <origin xyz="-0.061355 0 -0.33647" rpy="0 0 1.570796"/>
         <geometry>
-          <mesh filename="file://$(arg dae_file)" scale="1 0.964 1"/>
+          <mesh filename="file://$(arg dae_file)" scale="1 1 1"/>
         </geometry>
         <material name="black.001"/>
       </visual>
       <collision name="chassis_collision">
-        <origin xyz="0.058756 -0.03046 0.325149" rpy="1.570796 0 -3.141593"/>
+        <origin xyz="0.039687 -0.03046 0.350609" rpy="1.570796 0 -3.141593"/>
         <geometry>
-          <mesh filename="package://dbw_mkz_description/meshes/body_collision.stl" scale="0.000965 0.001 0.001"/>
+          <mesh filename="package://dbw_mkz_description/meshes/body_collision.stl" scale="0.001 0.001 0.001"/>
         </geometry>
       </collision>
@@ -46,7 +46,7 @@
       </inertial>
       <visual name="wheel_fl_visual">
-        <origin xyz="0 0 0.0385" rpy="-1.570796 -1.570796 0"/>
+        <origin xyz="-0.0026 0 0.032213" rpy="-1.570796 1.570796 0"/>
         <geometry>
-          <mesh filename="package://dbw_mkz_description/meshes/fusion/wheel.dae" scale="0.01 0.01 0.01"/>
+          <mesh filename="package://dbw_mkz_description/meshes/mondeo_15/wheel.dae" scale="0.01 0.01 0.01"/>
         </geometry>
         <material name="carpaint_002"/>
@@ -66,7 +66,7 @@
       </inertial>
       <visual name="wheel_fr_visual">
-        <origin xyz="0 0 -0.043777" rpy="-1.570796 1.570796 0"/>
+        <origin xyz="-0.0026 0 -0.035355" rpy="-1.570796 -1.570796 0"/>
         <geometry>
-          <mesh filename="package://dbw_mkz_description/meshes/fusion/wheel.dae" scale="0.01 0.01 0.01"/>
+          <mesh filename="package://dbw_mkz_description/meshes/mondeo_15/wheel.dae" scale="0.01 0.01 0.01"/>
         </geometry>
         <material name="carpaint_002.001"/>
@@ -86,7 +86,7 @@
       </inertial>
       <visual name="wheel_rl_visual">
-        <origin xyz="0 0 0.017382" rpy="-1.570796 -1.570796 0"/>
+        <origin xyz="0.0026 0 0.010943" rpy="-1.570796 1.570796 0"/>
         <geometry>
-          <mesh filename="package://dbw_mkz_description/meshes/fusion/wheel.dae" scale="0.01 0.01 0.01"/>
+          <mesh filename="package://dbw_mkz_description/meshes/mondeo_15/wheel.dae" scale="0.01 0.01 0.01"/>
         </geometry>
         <material name="carpaint_002.003"/>
@@ -106,7 +106,7 @@
       </inertial>
       <visual name="wheel_rr_visual">
-        <origin xyz="0 0 -0.019214" rpy="-1.570796 1.570796 0"/>
+        <origin xyz="0.0026 0 -0.010783" rpy="-1.570796 -1.570796 0"/>
         <geometry>
-          <mesh filename="package://dbw_mkz_description/meshes/fusion/wheel.dae" scale="0.01 0.01 0.01"/>
+          <mesh filename="package://dbw_mkz_description/meshes/mondeo_15/wheel.dae" scale="0.01 0.01 0.01"/>
         </geometry>
         <material name="carpaint_002.002"/>

Commit message: Restructured joints in URDF models.

File: dbw_mkz_description/urdf/fusion_13_structure.urdf.xacro (robot description, xacro)
@@ -7,17 +7,17 @@
     <link name="base_link">
       <inertial>
-        <origin xyz="0 0 0.25" rpy="0 0 0"/>
+        <origin xyz="1.4225 0 0.25" rpy="0 0 0"/>
         <mass value="1500.0"/>
         <inertia ixx="1000.0" ixy="0" ixz="0" iyy="1000.0" iyz="0" izz="1000.0"/>
       </inertial>
       <visual name="chassis">
-        <origin xyz="-0.045056 0 -0.373676" rpy="0 0 1.570796"/>
+        <origin xyz="1.3641 0 -0.373676" rpy="0 0 1.570796"/>
         <geometry>
-          <mesh filename="file://$(arg dae_file)" scale="1 0.964 1"/>
+          <mesh filename="file://$(arg dae_file)" scale="1 0.97 1"/>
         </geometry>
         <material name="black.001"/>
       </visual>
       <collision name="chassis_collision">
-        <origin xyz="0.058756 -0.03046 0.325149" rpy="1.570796 0 -3.141593"/>
+        <origin xyz="1.51 -0.03046 0.325149" rpy="1.570796 0 -3.141593"/>
         <geometry>
           <mesh filename="package://dbw_mkz_description/meshes/body_collision.stl" scale="0.000965 0.001 0.001"/>
@@ -125,5 +125,5 @@
     </joint>
     <joint name="steer_fl" type="revolute">
-      <origin xyz="1.435054 0.817 0.33" rpy="0 0 0"/>
+      <origin xyz="2.85 0.79121 0" rpy="0 0 0"/>
       <parent link="base_link"/>
       <child link="steer_fl"/>
@@ -132,5 +132,5 @@
     </joint>
     <joint name="steer_fr" type="revolute">
-      <origin xyz="1.43505 -0.815 0.33" rpy="0 0 0"/>
+      <origin xyz="2.85 -0.79121 0" rpy="0 0 0"/>
       <parent link="base_link"/>
       <child link="steer_fr"/>
@@ -139,5 +139,5 @@
     </joint>
     <joint name="wheel_fl" type="continuous">
-      <origin xyz="-0.012654 -0.0295 -0.33" rpy="1.570796 0 -3.141593"/>
+      <origin xyz="0 0 0" rpy="1.570796 0 -3.141593"/>
       <parent link="steer_fl"/>
       <child link="wheel_fl"/>
@@ -146,5 +146,5 @@
     </joint>
     <joint name="wheel_fr" type="continuous">
-      <origin xyz="-0.01265 0.0275 -0.33" rpy="1.570796 0 -3.141593"/>
+      <origin xyz="0 0 0" rpy="1.570796 0 -3.141593"/>
       <parent link="steer_fr"/>
       <child link="wheel_fr"/>
@@ -153,5 +153,5 @@
     </joint>
     <joint name="wheel_rl" type="continuous">
-      <origin xyz="-1.4224 0.808618 0" rpy="1.570796 0 -3.141593"/>
+      <origin xyz="0 0.7874 0" rpy="1.570796 0 -3.141593"/>
       <parent link="base_link"/>
       <child link="wheel_rl"/>
@@ -160,5 +160,5 @@
     </joint>
     <joint name="wheel_rr" type="continuous">
-      <origin xyz="-1.4224 -0.808 0" rpy="1.570796 0 -3.141593"/>
+      <origin xyz="0 -0.7874 0" rpy="1.570796 0 -3.141593"/>
       <parent link="base_link"/>
       <child link="wheel_rr"/>

File: dbw_mkz_description/urdf/mkz_13_structure.urdf.xacro (robot description, xacro)
@@ -7,17 +7,17 @@
     <link name="base_link">
       <inertial>
-        <origin xyz="0 0 0.25" rpy="0 0 0"/>
+        <origin xyz="1.4225 0 0.25" rpy="0 0 0"/>
         <mass value="1500.0"/>
         <inertia ixx="1000.0" ixy="0" ixz="0" iyy="1000.0" iyz="0" izz="1000.0"/>
       </inertial>
       <visual name="chassis">
-        <origin xyz="-0.058415 0 -0.33" rpy="0 0 1.570796"/>
+        <origin xyz="1.3641 0 -0.33" rpy="0 0 1.570796"/>
         <geometry>
-          <mesh filename="file://$(arg dae_file)" scale="0.394 0.394 0.394"/>
+          <mesh filename="file://$(arg dae_file)" scale="0.38 0.394 0.394"/>
         </geometry>
         <material name="black.001"/>
       </visual>
       <collision name="chassis_collision">
-        <origin xyz="0.084967 -0.03046 0.350609" rpy="1.570796 0 -3.141593"/>
+        <origin xyz="1.51 -0.03046 0.350609" rpy="1.570796 0 -3.141593"/>
         <geometry>
           <mesh filename="package://dbw_mkz_description/meshes/body_collision.stl" scale="0.001 0.001 0.001"/>
@@ -81,5 +81,5 @@
     <link name="wheel_rl">
       <inertial>
-        <origin xyz="0 0 -0.021117" rpy="0 3.141593 0"/>
+        <origin xyz="0 0 0" rpy="0 3.141593 0"/>
         <mass value="10.0"/>
         <inertia ixx="0.305583" ixy="0" ixz="0" iyy="0.305583" iyz="0" izz="0.5445"/>
@@ -101,5 +101,5 @@
     <link name="wheel_rr">
       <inertial>
-        <origin xyz="0 0 0.0205" rpy="0 3.141593 0"/>
+        <origin xyz="0 0 0" rpy="0 3.141593 0"/>
         <mass value="10.0"/>
         <inertia ixx="0.305583" ixy="0" ixz="0" iyy="0.305583" iyz="0" izz="0.5445"/>
@@ -125,5 +125,5 @@
     </joint>
     <joint name="steer_fl" type="revolute">
-      <origin xyz="1.435054 0.817 0.33" rpy="0 0 0"/>
+      <origin xyz="2.85 0.79121 0.0" rpy="0 0 0"/>
       <parent link="base_link"/>
       <child link="steer_fl"/>
@@ -132,5 +132,5 @@
     </joint>
     <joint name="steer_fr" type="revolute">
-      <origin xyz="1.43505 -0.815 0.33" rpy="0 0 0"/>
+      <origin xyz="2.85 -0.79121 0.0" rpy="0 0 0"/>
       <parent link="base_link"/>
       <child link="steer_fr"/>
@@ -139,5 +139,5 @@
     </joint>
     <joint name="wheel_fl" type="continuous">
-      <origin xyz="-0.012654 -0.0295 -0.33" rpy="1.570796 0 -3.141593"/>
+      <origin xyz="0 0 0" rpy="1.570796 0 -3.141593"/>
       <parent link="steer_fl"/>
       <child link="wheel_fl"/>
@@ -146,5 +146,5 @@
     </joint>
     <joint name="wheel_fr" type="continuous">
-      <origin xyz="-0.01265 0.0275 -0.33" rpy="1.570796 0 -3.141593"/>
+      <origin xyz="0 0 0" rpy="1.570796 0 -3.141593"/>
       <parent link="steer_fr"/>
       <child link="wheel_fr"/>
@@ -153,5 +153,5 @@
     </joint>
     <joint name="wheel_rl" type="continuous">
-      <origin xyz="-1.4224 0.808618 0" rpy="1.570796 0 -3.141593"/>
+      <origin xyz="0 0.7874 0" rpy="1.570796 0 -3.141593"/>
       <parent link="base_link"/>
       <child link="wheel_rl"/>
@@ -160,5 +160,5 @@
     </joint>
     <joint name="wheel_rr" type="continuous">
-      <origin xyz="-1.4224 -0.808 0" rpy="1.570796 0 -3.141593"/>
+      <origin xyz="0 -0.7874 0" rpy="1.570796 0 -3.141593"/>
       <parent link="base_link"/>
       <child link="wheel_rr"/>

File: dbw_mkz_description/urdf/mkz_17_structure.urdf.xacro (robot description, xacro)
@@ -7,17 +7,17 @@
     <link name="base_link">
       <inertial>
-        <origin xyz="0 0 0.25" rpy="0 0 0"/>
+        <origin xyz="1.4225 0 0.25" rpy="0 0 0"/>
         <mass value="1500.0"/>
         <inertia ixx="1000.0" ixy="0" ixz="0" iyy="1000.0" iyz="0" izz="1000.0"/>
       </inertial>
       <visual name="chassis">
-        <origin xyz="-0.032498 0 -0.371498" rpy="0 0 1.570796"/>
+        <origin xyz="1.39 0 -0.371498" rpy="0 0 1.570796"/>
         <geometry>
-          <mesh filename="file://$(arg dae_file)" scale="1 0.964 1"/>
+          <mesh filename="file://$(arg dae_file)" scale="1 0.97 1"/>
         </geometry>
         <material name="black.001"/>
       </visual>
       <collision name="chassis_collision">
-        <origin xyz="0.054381 -0.019748 0.332734" rpy="1.570796 0 -3.141593"/>
+        <origin xyz="1.4768 -0.019748 0.332734" rpy="1.570796 0 -3.141593"/>
         <geometry>
           <mesh filename="package://dbw_mkz_description/meshes/body_collision.stl" scale="0.001 0.001 0.001"/>
@@ -27,5 +27,5 @@
     <link name="steer_fl">
       <inertial>
-        <origin xyz="-0.013054 -0.0295 0" rpy="0 0 0"/>
+        <origin xyz="0 0 0" rpy="0 0 0"/>
         <mass value="1.0"/>
         <inertia ixx="0.037227" ixy="0" ixz="0" iyy="0.04" iyz="0" izz="0.06"/>
@@ -34,5 +34,5 @@
     <link name="steer_fr">
       <inertial>
-        <origin xyz="-0.01305 0.0275 0" rpy="0 0 0"/>
+        <origin xyz="0 0 0" rpy="0 0 0"/>
         <mass value="1.0"/>
         <inertia ixx="0.037227" ixy="0" ixz="0" iyy="0.04" iyz="0" izz="0.06"/>
@@ -125,5 +125,5 @@
     </joint>
     <joint name="steer_fl" type="revolute">
-      <origin xyz="1.435054 0.817 0.33" rpy="0 0 0"/>
+      <origin xyz="2.85 0.79712 0" rpy="0 0 0"/>
       <parent link="base_link"/>
       <child link="steer_fl"/>
@@ -132,5 +132,5 @@
     </joint>
     <joint name="steer_fr" type="revolute">
-      <origin xyz="1.43505 -0.815 0.33" rpy="0 0 0"/>
+      <origin xyz="2.85 -0.79712 0.0" rpy="0 0 0"/>
       <parent link="base_link"/>
       <child link="steer_fr"/>
@@ -139,5 +139,5 @@
     </joint>
     <joint name="wheel_fl" type="continuous">
-      <origin xyz="-0.012654 -0.0295 -0.33" rpy="1.570796 0 -3.141593"/>
+      <origin xyz="0 0 0" rpy="1.570796 0 -3.141593"/>
       <parent link="steer_fl"/>
       <child link="wheel_fl"/>
@@ -146,5 +146,5 @@
     </joint>
     <joint name="wheel_fr" type="continuous">
-      <origin xyz="-0.01265 0.0275 -0.33" rpy="1.570796 0 -3.141593"/>
+      <origin xyz="0 0 0" rpy="1.570796 0 -3.141593"/>
       <parent link="steer_fr"/>
       <child link="wheel_fr"/>
@@ -153,5 +153,5 @@
     </joint>
     <joint name="wheel_rl" type="continuous">
-      <origin xyz="-1.4224 0.808618 0" rpy="1.570796 0 -3.141593"/>
+      <origin xyz="0 0.7874 0" rpy="1.570796 0 -3.141593"/>
       <parent link="base_link"/>
       <child link="wheel_rl"/>
@@ -160,5 +160,5 @@
     </joint>
     <joint name="wheel_rr" type="continuous">
-      <origin xyz="-1.4224 -0.808 0" rpy="1.570796 0 -3.141593"/>
+      <origin xyz="0 -0.7874 0" rpy="1.570796 0 -3.141593"/>
       <parent link="base_link"/>
       <child link="wheel_rr"/>

File: dbw_mkz_description/urdf/mondeo_15_structure.urdf.xacro (robot description, xacro)
@@ -7,10 +7,10 @@
     <link name="base_link">
       <inertial>
-        <origin xyz="0 0 0.25" rpy="0 0 0"/>
+        <origin xyz="1.4225 0 0.25" rpy="0 0 0"/>
         <mass value="1500.0"/>
         <inertia ixx="1000.0" ixy="0" ixz="0" iyy="1000.0" iyz="0" izz="1000.0"/>
       </inertial>
       <visual name="chassis">
-        <origin xyz="-0.061355 0 -0.33647" rpy="0 0 1.570796"/>
+        <origin xyz="1.361 0 -0.33647" rpy="0 0 1.570796"/>
         <geometry>
           <mesh filename="file://$(arg dae_file)" scale="1 1 1"/>
@@ -19,5 +19,5 @@
       </visual>
       <collision name="chassis_collision">
-        <origin xyz="0.039687 -0.03046 0.350609" rpy="1.570796 0 -3.141593"/>
+        <origin xyz="1.4621 -0.03046 0.350609" rpy="1.570796 0 -3.141593"/>
         <geometry>
           <mesh filename="package://dbw_mkz_description/meshes/body_collision.stl" scale="0.001 0.001 0.001"/>
@@ -27,5 +27,5 @@
     <link name="steer_fl">
       <inertial>
-        <origin xyz="-0.013054 -0.0295 0" rpy="0 0 0"/>
+        <origin xyz="0 0 0" rpy="0 0 0"/>
         <mass value="1.0"/>
         <inertia ixx="0.037227" ixy="0" ixz="0" iyy="0.04" iyz="0" izz="0.06"/>
@@ -34,5 +34,5 @@
     <link name="steer_fr">
       <inertial>
-        <origin xyz="-0.01305 0.0275 0" rpy="0 0 0"/>
+        <origin xyz="0 0 0" rpy="0 0 0"/>
         <mass value="1.0"/>
         <inertia ixx="0.037227" ixy="0" ixz="0" iyy="0.04" iyz="0" izz="0.06"/>
@@ -125,5 +125,5 @@
     </joint>
     <joint name="steer_fl" type="revolute">
-      <origin xyz="1.435054 0.817 0.33" rpy="0 0 0"/>
+      <origin xyz="2.85 0.79121 0" rpy="0 0 0"/>
       <parent link="base_link"/>
       <child link="steer_fl"/>
@@ -132,5 +132,5 @@
     </joint>
     <joint name="steer_fr" type="revolute">
-      <origin xyz="1.43505 -0.815 0.33" rpy="0 0 0"/>
+      <origin xyz="2.85 -0.79121 0" rpy="0 0 0"/>
       <parent link="base_link"/>
       <child link="steer_fr"/>
@@ -139,5 +139,5 @@
     </joint>
     <joint name="wheel_fl" type="continuous">
-      <origin xyz="-0.012654 -0.0295 -0.33" rpy="1.570796 0 -3.141593"/>
+      <origin xyz="0 0 0" rpy="1.570796 0 -3.141593"/>
       <parent link="steer_fl"/>
       <child link="wheel_fl"/>
@@ -146,5 +146,5 @@
     </joint>
     <joint name="wheel_fr" type="continuous">
-      <origin xyz="-0.01265 0.0275 -0.33" rpy="1.570796 0 -3.141593"/>
+      <origin xyz="0 0 0" rpy="1.570796 0 -3.141593"/>
       <parent link="steer_fr"/>
       <child link="wheel_fr"/>
@@ -153,5 +153,5 @@
     </joint>
     <joint name="wheel_rl" type="continuous">
-      <origin xyz="-1.4224 0.808618 0" rpy="1.570796 0 -3.141593"/>
+      <origin xyz="0 0.7874 0" rpy="1.570796 0 -3.141593"/>
       <parent link="base_link"/>
       <child link="wheel_rl"/>
@@ -160,5 +160,5 @@
     </joint>
     <joint name="wheel_rr" type="continuous">
-      <origin xyz="-1.4224 -0.808 0" rpy="1.570796 0 -3.141593"/>
+      <origin xyz="0 -0.7874 0" rpy="1.570796 0 -3.141593"/>
       <parent link="base_link"/>
       <child link="wheel_rr"/>
