Commit message: Changes names of joints to be different from links
Gazebo 11 doesn't let joint names and link names be the same, which was allowed in earlier versions

File: dbw_mkz_description/urdf/f150_14_structure.urdf.xacro (robot description, xacro)
@@ -30,5 +30,5 @@
       </inertial>
     </link>
-    <joint name="wheel_${name}" type="continuous" >
+    <joint name="wheel_${name}_joint" type="continuous" >
       <parent link="base_link" />
       <child link="wheel_${name}" />
@@ -64,5 +64,5 @@
       </inertial>
     </link>
-    <joint name="steer_${name}" type="revolute" >
+    <joint name="steer_${name}_joint" type="revolute" >
       <parent link="base_link" />
       <child link="steer_${name}" />
@@ -71,5 +71,5 @@
       <limit upper="0.6" lower="-0.6" effort="0.0" velocity="0.0" />
     </joint>
-    <joint name="wheel_${name}" type="continuous" >
+    <joint name="wheel_${name}_joint" type="continuous" >
       <parent link="steer_${name}" />
       <child link="wheel_${name}" />
@@ -107,10 +107,10 @@
     </visual>
   </link>
-  <joint name="base_link" type="fixed" >
+  <joint name="base_link_joint" type="fixed" >
     <parent link="base_footprint" />
     <child link="base_link" />
     <origin xyz="${half_wheelbase} 0 ${wheel_radius}" rpy="0 0 0" />
   </joint>
-  <joint name="hood_logo" type="fixed" >
+  <joint name="hood_logo_joint" type="fixed" >
     <parent link="base_link" />
     <child link="hood_logo" />

File: dbw_mkz_description/urdf/fusion_13_structure.urdf.xacro (robot description, xacro)
@@ -119,10 +119,10 @@
       </collision>
     </link>
-    <joint name="base_link" type="fixed">
+    <joint name="base_link_joint" type="fixed">
       <origin xyz="0 0 0.33" rpy="0 0 0"/>
       <parent link="base_footprint"/>
       <child link="base_link"/>
     </joint>
-    <joint name="steer_fl" type="revolute">
+    <joint name="steer_fl_joint" type="revolute">
       <origin xyz="2.85 0.79121 0" rpy="0 0 0"/>
       <parent link="base_link"/>
@@ -131,5 +131,5 @@
       <limit lower="-0.6" upper="0.6" effort="0" velocity="0"/>
     </joint>
-    <joint name="steer_fr" type="revolute">
+    <joint name="steer_fr_joint" type="revolute">
       <origin xyz="2.85 -0.79121 0" rpy="0 0 0"/>
       <parent link="base_link"/>
@@ -138,5 +138,5 @@
       <limit lower="-0.6" upper="0.6" effort="0" velocity="0"/>
     </joint>
-    <joint name="wheel_fl" type="continuous">
+    <joint name="wheel_fl_joint" type="continuous">
       <origin xyz="0 0 0" rpy="1.570796 0 -3.141593"/>
       <parent link="steer_fl"/>
@@ -145,5 +145,5 @@
       <limit effort="0" velocity="22.0"/>
     </joint>
-    <joint name="wheel_fr" type="continuous">
+    <joint name="wheel_fr_joint" type="continuous">
       <origin xyz="0 0 0" rpy="1.570796 0 -3.141593"/>
       <parent link="steer_fr"/>
@@ -152,5 +152,5 @@
       <limit effort="0" velocity="22.0"/>
     </joint>
-    <joint name="wheel_rl" type="continuous">
+    <joint name="wheel_rl_joint" type="continuous">
       <origin xyz="0 0.7874 0" rpy="1.570796 0 -3.141593"/>
       <parent link="base_link"/>
@@ -159,5 +159,5 @@
       <limit effort="5000.0" velocity="22.0"/>
     </joint>
-    <joint name="wheel_rr" type="continuous">
+    <joint name="wheel_rr_joint" type="continuous">
       <origin xyz="0 -0.7874 0" rpy="1.570796 0 -3.141593"/>
       <parent link="base_link"/>

File: dbw_mkz_description/urdf/mkz_13_structure.urdf.xacro (robot description, xacro)
@@ -119,10 +119,10 @@
       </collision>
     </link>
-    <joint name="base_link" type="fixed">
+    <joint name="base_link_joint" type="fixed">
       <origin xyz="0 0 0.33" rpy="0 0 0"/>
       <parent link="base_footprint"/>
       <child link="base_link"/>
     </joint>
-    <joint name="steer_fl" type="revolute">
+    <joint name="steer_fl_joint" type="revolute">
       <origin xyz="2.85 0.79121 0.0" rpy="0 0 0"/>
       <parent link="base_link"/>
@@ -131,5 +131,5 @@
       <limit lower="-0.6" upper="0.6" effort="0" velocity="0"/>
     </joint>
-    <joint name="steer_fr" type="revolute">
+    <joint name="steer_fr_joint" type="revolute">
       <origin xyz="2.85 -0.79121 0.0" rpy="0 0 0"/>
       <parent link="base_link"/>
@@ -138,5 +138,5 @@
       <limit lower="-0.6" upper="0.6" effort="0" velocity="0"/>
     </joint>
-    <joint name="wheel_fl" type="continuous">
+    <joint name="wheel_fl_joint" type="continuous">
       <origin xyz="0 0 0" rpy="1.570796 0 -3.141593"/>
       <parent link="steer_fl"/>
@@ -145,5 +145,5 @@
       <limit effort="0" velocity="22.0"/>
     </joint>
-    <joint name="wheel_fr" type="continuous">
+    <joint name="wheel_fr_joint" type="continuous">
       <origin xyz="0 0 0" rpy="1.570796 0 -3.141593"/>
       <parent link="steer_fr"/>
@@ -152,5 +152,5 @@
       <limit effort="0" velocity="22.0"/>
     </joint>
-    <joint name="wheel_rl" type="continuous">
+    <joint name="wheel_rl_joint" type="continuous">
       <origin xyz="0 0.7874 0" rpy="1.570796 0 -3.141593"/>
       <parent link="base_link"/>
@@ -159,5 +159,5 @@
       <limit effort="5000.0" velocity="22.0"/>
     </joint>
-    <joint name="wheel_rr" type="continuous">
+    <joint name="wheel_rr_joint" type="continuous">
       <origin xyz="0 -0.7874 0" rpy="1.570796 0 -3.141593"/>
       <parent link="base_link"/>

File: dbw_mkz_description/urdf/mkz_17_structure.urdf.xacro (robot description, xacro)
@@ -119,10 +119,10 @@
       </collision>
     </link>
-    <joint name="base_link" type="fixed">
+    <joint name="base_link_joint" type="fixed">
       <origin xyz="0 0 0.33" rpy="0 0 0"/>
       <parent link="base_footprint"/>
       <child link="base_link"/>
     </joint>
-    <joint name="steer_fl" type="revolute">
+    <joint name="steer_fl_joint" type="revolute">
       <origin xyz="2.85 0.79712 0" rpy="0 0 0"/>
       <parent link="base_link"/>
@@ -131,5 +131,5 @@
       <limit lower="-0.6" upper="0.6" effort="0" velocity="0"/>
     </joint>
-    <joint name="steer_fr" type="revolute">
+    <joint name="steer_fr_joint" type="revolute">
       <origin xyz="2.85 -0.79712 0.0" rpy="0 0 0"/>
       <parent link="base_link"/>
@@ -138,5 +138,5 @@
       <limit lower="-0.6" upper="0.6" effort="0" velocity="0"/>
     </joint>
-    <joint name="wheel_fl" type="continuous">
+    <joint name="wheel_fl_joint" type="continuous">
       <origin xyz="0 0 0" rpy="1.570796 0 -3.141593"/>
       <parent link="steer_fl"/>
@@ -145,5 +145,5 @@
       <limit effort="0" velocity="22.0"/>
     </joint>
-    <joint name="wheel_fr" type="continuous">
+    <joint name="wheel_fr_joint" type="continuous">
       <origin xyz="0 0 0" rpy="1.570796 0 -3.141593"/>
       <parent link="steer_fr"/>
@@ -152,5 +152,5 @@
       <limit effort="0" velocity="22.0"/>
     </joint>
-    <joint name="wheel_rl" type="continuous">
+    <joint name="wheel_rl_joint" type="continuous">
       <origin xyz="0 0.7874 0" rpy="1.570796 0 -3.141593"/>
       <parent link="base_link"/>
@@ -159,5 +159,5 @@
       <limit effort="5000.0" velocity="22.0"/>
     </joint>
-    <joint name="wheel_rr" type="continuous">
+    <joint name="wheel_rr_joint" type="continuous">
       <origin xyz="0 -0.7874 0" rpy="1.570796 0 -3.141593"/>
       <parent link="base_link"/>

File: dbw_mkz_description/urdf/mondeo_15_structure.urdf.xacro (robot description, xacro)
@@ -119,10 +119,10 @@
       </collision>
     </link>
-    <joint name="base_link" type="fixed">
+    <joint name="base_link_joint" type="fixed">
       <origin xyz="0 0 0.33" rpy="0 0 0"/>
       <parent link="base_footprint"/>
       <child link="base_link"/>
     </joint>
-    <joint name="steer_fl" type="revolute">
+    <joint name="steer_fl_joint" type="revolute">
       <origin xyz="2.85 0.79121 0" rpy="0 0 0"/>
       <parent link="base_link"/>
@@ -131,5 +131,5 @@
       <limit lower="-0.6" upper="0.6" effort="0" velocity="0"/>
     </joint>
-    <joint name="steer_fr" type="revolute">
+    <joint name="steer_fr_joint" type="revolute">
       <origin xyz="2.85 -0.79121 0" rpy="0 0 0"/>
       <parent link="base_link"/>
@@ -138,5 +138,5 @@
       <limit lower="-0.6" upper="0.6" effort="0" velocity="0"/>
     </joint>
-    <joint name="wheel_fl" type="continuous">
+    <joint name="wheel_fl_joint" type="continuous">
       <origin xyz="0 0 0" rpy="1.570796 0 -3.141593"/>
       <parent link="steer_fl"/>
@@ -145,5 +145,5 @@
       <limit effort="0" velocity="22.0"/>
     </joint>
-    <joint name="wheel_fr" type="continuous">
+    <joint name="wheel_fr_joint" type="continuous">
       <origin xyz="0 0 0" rpy="1.570796 0 -3.141593"/>
       <parent link="steer_fr"/>
@@ -152,5 +152,5 @@
       <limit effort="0" velocity="22.0"/>
     </joint>
-    <joint name="wheel_rl" type="continuous">
+    <joint name="wheel_rl_joint" type="continuous">
       <origin xyz="0 0.7874 0" rpy="1.570796 0 -3.141593"/>
       <parent link="base_link"/>
@@ -159,5 +159,5 @@
       <limit effort="5000.0" velocity="22.0"/>
     </joint>
-    <joint name="wheel_rr" type="continuous">
+    <joint name="wheel_rr_joint" type="continuous">
       <origin xyz="0 -0.7874 0" rpy="1.570796 0 -3.141593"/>
       <parent link="base_link"/>
